Commit message: Added code and launch files for Final Project

File: diff_drive_bot/description/robot_core.xacro (robot description, xacro)
@@ -29,5 +29,5 @@
 				<box size="0.3 0.3 0.15"/>
 			</geometry>
-			<material name="white"/>
+			<material name="orange"/>
 		</visual>
 		<collision>
@@ -41,4 +41,7 @@
 		</xacro:inertial_box>
 	</link>
+	<gazebo reference="chassis">
+		<material>Gazebo/Orange</material>
+	</gazebo>
 <!-- Left Wheel Link -->
 	<joint name="left_wheel_joint" type="continuous">
@@ -64,4 +67,7 @@
 		</xacro:inertial_cylinder>
 	</link>
+	<gazebo reference="left_wheel">
+		<material>Gazebo/Blue</material>
+	</gazebo>
 <!-- Right Wheel Link -->
 	<joint name="right_wheel_joint" type="continuous">
@@ -87,4 +93,7 @@
 		</xacro:inertial_cylinder>
 	</link>
+	<gazebo reference="right_wheel">
+		<material>Gazebo/Blue</material>
+	</gazebo>
 <!-- Caster Wheel Link -->
 	<joint name="caster_wheel_joint" type="fixed">
@@ -109,3 +118,8 @@
 		</xacro:inertial_sphere>
 	</link>
+	<gazebo reference="caster_wheel">
+		<material>Gazebo/Black</material>
+		<mu1 value="0.001"/>
+		<mu2 value="0.001"/>
+	</gazebo>
 </robot>
